File: accessController.sch (KiCad schematic (older format))
At the start: 33 parts, among them J1 220V AC POWER, J2 Load, J3 Screw_Terminal_01x02, J4 GPIO, J5 Conn_01x04, K1 HJR-3FF-5VDC-S-Z, Q1 BSS138, SW1 SW_Push, SW2 SW_Push, U1 ACS712xLCTR-20A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

Commit message: Update
Parts:
- J1: value 220V AC POWER -> DG129-5.0-03P-14-00AH
- J2: value Load -> DG129-5.0-03P-14-00AH
- J3: value Screw_Terminal_01x02 -> DG129-5.0-02P-14-00AH
Other:
- note added: "220V AC"
- note added: "Current"
- note added: "Load"
Changed lines of the file:
@@
 P 1300 2250
 F 0 "J1" H 1218 1925 50  0000 C CNN
-F 1 "220V AC POWER" H 1218 2016 50  0000 C CNN
+F 1 "DG129-5.0-03P-14-00AH" H 1218 2016 50  0000 C CNN
 F 2 "TerminalBlock:TerminalBlock_Altech_AK300-3_P5.00mm" H 1300 2250 50  0001 C CNN
 F 3 "~" H 1300 2250 50  0001 C CNN
@@
 P 1350 3450
 F 0 "J2" H 1268 3125 50  0000 C CNN
-F 1 "Load" H 1268 3216 50  0000 C CNN
+F 1 "DG129-5.0-03P-14-00AH" H 1268 3216 50  0000 C CNN
 F 2 "TerminalBlock:TerminalBlock_Altech_AK300-3_P5.00mm" H 1350 3450 50  0001 C CNN
 F 3 "~" H 1350 3450 50  0001 C CNN
@@
 P 1500 6900
 F 0 "J3" H 1418 6575 50  0000 C CNN
-F 1 "Screw_Terminal_01x02" H 1418 6666 50  0000 C CNN
+F 1 "DG129-5.0-02P-14-00AH" H 1418 6666 50  0000 C CNN
 F 2 "TerminalBlock:TerminalBlock_Altech_AK300-2_P5.00mm" H 1500 6900 50  0001 C CNN
 F 3 "~" H 1500 6900 50  0001 C CNN
@@
 Wire Wire Line
 	6300 4000 7650 4000
+Text Notes 850  2300 0    50   ~ 0
+220V AC
+Text Notes 1050 3500 0    50   ~ 0
+Load
+Text Notes 1100 6900 0    50   ~ 0
+Current
 $EndSCHEMATC
